File: PMS5003S_MOUNT.kicad_pcb (KiCad board)
At the start: 2 copper layers, 90 x 90 mm, 9 parts, among them J1 CONN_MCU, J2 CONN_PMS, U1 USB_PCB

Commit message: update,
Parts:
- moved R1 74.7 mm to (21.0, 11.0), turned to 270 degrees
- moved R2 66.5 mm to (21.0, 16.0), turned to 90 degrees
- moved J1 55.8 mm to (26.0, 11.0)
- moved J2 39.4 mm to (45.0, 8.00), turned to 90 degrees
Other:
- outline, holes or cut-outs redrawn
Changed lines of the file:
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@@
   )
   (module Connector_PinHeader_2.54mm:PinHeader_1x06_P2.54mm_Vertical (layer F.Cu)
-    (at 75.475001 36.825001)
+    (at 26 11)
     (descr "Through hole straight pin header, 1x06, 2.54mm pitch, single row")
     (tags "Through hole pin header THT 1x06 2.54mm single row")
@@
   )
   (module Connector_PinHeader_2.54mm:PinHeader_1x08_P2.54mm_Vertical (layer F.Cu)
-    (at 71.825001 36.825001)
+    (at 45 8 90)
     (descr "Through hole straight pin header, 1x08, 2.54mm pitch, single row")
     (tags "Through hole pin header THT 1x08 2.54mm single row")
-    (fp_text reference J2 (at 0 -2.33) (layer F.SilkS)
-      (effects (font (size 1 1) (thickness 0.15)))
-    )
-    (fp_text value CONN_PMS (at 0 20.11) (layer F.Fab)
+    (fp_text reference J2 (at 0 -2.33 90) (layer F.SilkS)
+      (effects (font (size 1 1) (thickness 0.15)))
+    )
+    (fp_text value CONN_PMS (at 0 20.11 90) (layer F.Fab)
       (effects (font (size 1 1) (thickness 0.15)))
     )
@@
     (fp_line (start 1.8 19.55) (end 1.8 -1.8) (layer F.CrtYd) (width 0.05))
     (fp_line (start 1.8 -1.8) (end -1.8 -1.8) (layer F.CrtYd) (width 0.05))
-    (fp_text user %R (at 0 8.89 90) (layer F.Fab)
-      (effects (font (size 1 1) (thickness 0.15)))
-    )
-    (pad 1 thru_hole rect (at 0 0) (size 1.7 1.7) (drill 1) (layers *.Cu *.Mask)
+    (fp_text user %R (at 0 8.89 180) (layer F.Fab)
+      (effects (font (size 1 1) (thickness 0.15)))
+    )
+    (pad 1 thru_hole rect (at 0 0 90) (size 1.7 1.7) (drill 1) (layers *.Cu *.Mask)
       (net 8 +5V))
-    (pad 2 thru_hole oval (at 0 2.54) (size 1.7 1.7) (drill 1) (layers *.Cu *.Mask)
+    (pad 2 thru_hole oval (at 0 2.54 90) (size 1.7 1.7) (drill 1) (layers *.Cu *.Mask)
       (net 9 GND))
-    (pad 3 thru_hole oval (at 0 5.08) (size 1.7 1.7) (drill 1) (layers *.Cu *.Mask)
+    (pad 3 thru_hole oval (at 0 5.08 90) (size 1.7 1.7) (drill 1) (layers *.Cu *.Mask)
       (net 6 /SEN_SET))
-    (pad 4 thru_hole oval (at 0 7.62) (size 1.7 1.7) (drill 1) (layers *.Cu *.Mask)
+    (pad 4 thru_hole oval (at 0 7.62 90) (size 1.7 1.7) (drill 1) (layers *.Cu *.Mask)
       (net 10 /SEN_RXD))
-    (pad 5 thru_hole oval (at 0 10.16) (size 1.7 1.7) (drill 1) (layers *.Cu *.Mask)
+    (pad 5 thru_hole oval (at 0 10.16 90) (size 1.7 1.7) (drill 1) (layers *.Cu *.Mask)
       (net 11 /SEN_TXD))
-    (pad 6 thru_hole oval (at 0 12.7) (size 1.7 1.7) (drill 1) (layers *.Cu *.Mask)
+    (pad 6 thru_hole oval (at 0 12.7 90) (size 1.7 1.7) (drill 1) (layers *.Cu *.Mask)
       (net 7 /SEN_RESET))
-    (pad 7 thru_hole oval (at 0 15.24) (size 1.7 1.7) (drill 1) (layers *.Cu *.Mask)
+    (pad 7 thru_hole oval (at 0 15.24 90) (size 1.7 1.7) (drill 1) (layers *.Cu *.Mask)
       (net 12 "Net-(J2-Pad7)"))
-    (pad 8 thru_hole oval (at 0 17.78) (size 1.7 1.7) (drill 1) (layers *.Cu *.Mask)
+    (pad 8 thru_hole oval (at 0 17.78 90) (size 1.7 1.7) (drill 1) (layers *.Cu *.Mask)
       (net 13 "Net-(J2-Pad8)"))
     (model ${KISYS3DMOD}/Connector_PinHeader_2.54mm.3dshapes/PinHeader_1x08_P2.54mm_Vertical.wrl
@@
   )
   (module Resistor_SMD:R_0805_2012Metric_Pad1.15x1.40mm_HandSolder (layer F.Cu)
-    (at 79.175001 48.295001)
+    (at 21 16.025 90)
     (descr "Resistor SMD 0805 (2012 Metric), square (rectangular) end terminal, IPC_7351 nominal with elongated pad for handsoldering. (Body size source: https://docs.google.com/spreadsheets/d/1BsfQQcO9C6DZCsRaXUlFlo91Tg2WpOkGARC1WS5S8t0/edit?usp=sharing), generated with kicad-footprint-generator")
     (tags "resistor handsolder")
     (attr smd)
-    (fp_text reference R2 (at 0 -1.65) (layer F.SilkS)
-      (effects (font (size 1 1) (thickness 0.15)))
-    )
-    (fp_text value R103 (at 0 1.65) (layer F.Fab)
-      (effects (font (size 1 1) (thickness 0.15)))
-    )
-    (fp_text user %R (at 0 0) (layer F.Fab)
+    (fp_text reference R2 (at 0 -1.65 90) (layer F.SilkS)
+      (effects (font (size 1 1) (thickness 0.15)))
+    )
+    (fp_text value R103 (at 0 1.65 90) (layer F.Fab)
+      (effects (font (size 1 1) (thickness 0.15)))
+    )
+    (fp_text user %R (at 0 0 90) (layer F.Fab)
       (effects (font (size 0.5 0.5) (thickness 0.08)))
     )
@@
     (fp_line (start -1 -0.6) (end 1 -0.6) (layer F.Fab) (width 0.1))
     (fp_line (start -1 0.6) (end -1 -0.6) (layer F.Fab) (width 0.1))
-    (pad 2 smd roundrect (at 1.025 0) (size 1.15 1.4) (layers F.Cu F.Paste F.Mask) (roundrect_rratio 0.217391)
+    (pad 2 smd roundrect (at 1.025 0 90) (size 1.15 1.4) (layers F.Cu F.Paste F.Mask) (roundrect_rratio 0.217391)
       (net 5 +3V3))
-    (pad 1 smd roundrect (at -1.025 0) (size 1.15 1.4) (layers F.Cu F.Paste F.Mask) (roundrect_rratio 0.217391)
+    (pad 1 smd roundrect (at -1.025 0 90) (size 1.15 1.4) (layers F.Cu F.Paste F.Mask) (roundrect_rratio 0.217391)
       (net 7 /SEN_RESET))
     (model ${KISYS3DMOD}/Resistor_SMD.3dshapes/R_0805_2012Metric.wrl
@@
   )
   (module Resistor_SMD:R_0805_2012Metric_Pad1.15x1.40mm_HandSolder (layer F.Cu)
-    (at 91.385001 35.975001)
+    (at 21 10.975 270)
     (descr "Resistor SMD 0805 (2012 Metric), square (rectangular) end terminal, IPC_7351 nominal with elongated pad for handsoldering. (Body size source: https://docs.google.com/spreadsheets/d/1BsfQQcO9C6DZCsRaXUlFlo91Tg2WpOkGARC1WS5S8t0/edit?usp=sharing), generated with kicad-footprint-generator")
     (tags "resistor handsolder")
     (attr smd)
-    (fp_text reference R1 (at 0 -1.65) (layer F.SilkS)
-      (effects (font (size 1 1) (thickness 0.15)))
-    )
-    (fp_text value R103 (at 0 1.65) (layer F.Fab)
+    (fp_text reference R1 (at 0 -1.65 270) (layer F.SilkS)
+      (effects (font (size 1 1) (thickness 0.15)))
+    )
+    (fp_text value R103 (at 0 1.65 270) (layer F.Fab)
       (effects (font (size 1 1) (thickness 0.15)))
     )
@@
     (fp_line (start 1.85 -0.95) (end 1.85 0.95) (layer F.CrtYd) (width 0.05))
     (fp_line (start 1.85 0.95) (end -1.85 0.95) (layer F.CrtYd) (width 0.05))
-    (fp_text user %R (at 0 0) (layer F.Fab)
+    (fp_text user %R (at 0 0 270) (layer F.Fab)
       (effects (font (size 0.5 0.5) (thickness 0.08)))
     )
-    (pad 1 smd roundrect (at -1.025 0) (size 1.15 1.4) (layers F.Cu F.Paste F.Mask) (roundrect_rratio 0.217391)
+    (pad 1 smd roundrect (at -1.025 0 270) (size 1.15 1.4) (layers F.Cu F.Paste F.Mask) (roundrect_rratio 0.217391)
       (net 5 +3V3))
-    (pad 2 smd roundrect (at 1.025 0) (size 1.15 1.4) (layers F.Cu F.Paste F.Mask) (roundrect_rratio 0.217391)
+    (pad 2 smd roundrect (at 1.025 0 270) (size 1.15 1.4) (layers F.Cu F.Paste F.Mask) (roundrect_rratio 0.217391)
       (net 6 /SEN_SET))
     (model ${KISYS3DMOD}/Resistor_SMD.3dshapes/R_0805_2012Metric.wrl
@@
   (gr_line (start 25 70) (end 7 70) (layer Edge.Cuts) (width 0.15))
   (gr_line (start 27 58) (end 27 69) (layer Edge.Cuts) (width 0.15))
-  (gr_line (start 5 28) (end 5 8) (layer Edge.Cuts) (width 0.15))
+  (gr_line (start 5 28) (end 5 10) (layer Edge.Cuts) (width 0.15))
   (gr_line (start 5 45) (end 5 55) (layer Edge.Cuts) (width 0.15))
   (gr_line (start 6 56) (end 26 56) (layer Edge.Cuts) (width 0.15))

Commit message: update,
Parts:
- added C1: C106, Capacitor_SMD:C_0805_2012Metric_Pad1.15x1.40mm_HandSolder, F.Cu at (79.0, 35.0)
- added D1: LED_GREEN, LED_SMD:LED_0805_2012Metric_Pad1.15x1.40mm_HandSolder, F.Cu at (79.0, 32.0)
- added D2: LED_GREEN, LED_SMD:LED_0805_2012Metric_Pad1.15x1.40mm_HandSolder, F.Cu at (79.0, 28.0)
- added R3: R102, Resistor_SMD:R_0805_2012Metric_Pad1.15x1.40mm_HandSolder, F.Cu at (79.0, 25.0)
- added R4: R102, Resistor_SMD:R_0805_2012Metric_Pad1.15x1.40mm_HandSolder, F.Cu at (52.0, 37.0)
- moved J2 50.9 mm to (80.0, 45.0), turned to 270 degrees
- moved J1 42.8 mm to (52.0, 45.0), turned to 270 degrees
- moved R1 42.5 mm to (52.0, 40.0), turned to 180 degrees
- moved R2 35.3 mm to (47.0, 40.0), turned to 0 degrees
Connections:
- U1 pad 1: Net-(U1-Pad1) -> +5V
- U1 pad 4: Net-(U1-Pad4) -> GND
Other:
- outline, holes or cut-outs redrawn
- board text added: "PMS5003S"

Commit message: update,
Parts:
- removed REF** (x4): MountingHole_3.2mm_M3_DIN965, MountingHole:MountingHole_3.2mm_M3_DIN965
- removed U1: USB_PCB, footprint-lib.pretty:usb-PCB
- C1, R1, R2, R3, R4: moved to B.Cu
- J2: footprint Connector_PinHeader_2.54mm:PinHeader_1x08_P2.54mm_Vertical -> footprint-lib:PMS5003S
- moved R3 38.0 mm to (45.0, 42.0)
- moved D2 38.0 mm to (45.0, 45.0), turned to 0 degrees
- moved D1 35.5 mm to (45.0, 42.0), turned to 0 degrees
- moved C1 26.0 mm to (53.0, 35.5), turned to 180 degrees
- moved J1 19.6 mm to (33.7, 38.0), turned to 180 degrees
- moved R2 11.7 mm to (53.0, 30.0)
- moved R4 10.6 mm to (45.0, 45.0), turned to 0 degrees
- moved J2 8.77 mm to (74.0, 38.6), turned to 90 degrees
- moved R1 7.57 mm to (53.0, 32.5)
Connections:
- J2 pad 7: Net-(J2-Pad7) -> (no net)
- J2 pad 8: Net-(J2-Pad8) -> (no net)
Routing:
- net +3V3: track 0.00 -> 41.5 mm
- net GND: track 0.00 -> 30.1 mm
- net /SEN_RESET: track 0.00 -> 22.6 mm
- net /SEN_SET: track 0.00 -> 18.5 mm
- net +5V: track 0.00 -> 16.9 mm
- net /SEN_TXD: track 0.00 -> 9.59 mm
- net /SEN_RXD: track 0.00 -> 9.59 mm
- net Net-(D2-Pad2): vias 0 -> 1
- net Net-(D1-Pad2): vias 0 -> 1
Other:
- board outline removed
- board text removed: "PMS5003S"
