File: PMS5003S_MOUNT.sch (KiCad schematic (older format))
At the start: 5 parts, among them J1 CONN_MCU, J2 CONN_PMS, U1 USB_PCB

Commit message: update,
Parts:
- added C1: C106, Capacitor_SMD:C_0805_2012Metric_Pad1.15x1.40mm_HandSolder, symbol taobao-c:C106
- added D1, D2: LED_GREEN, LED_SMD:LED_0805_2012Metric_Pad1.15x1.40mm_HandSolder, symbol taobao-components:LED_GREEN
- added R3, R4: R102, Resistor_SMD:R_0805_2012Metric_Pad1.15x1.40mm_HandSolder, symbol taobao-r:R102
Connections:
- net +3V3: now also R4.1
- net +5V: now also U1.1 (VCC), C1.1, R3.1
- net GND: now also U1.4 (GND), C1.2, D1.1 (K), D2.1 (K)
- new net: D1.2 (A), R3.2
- new net: D2.2 (A), R4.2
Changed lines of the file:
@@
 $Descr A4 11693 8268
 encoding utf-8
-Sheet 1 1
+Sheet 1 2
 Title ""
 Date ""
@@
 U 1 1 5BC627DA
 P 2650 3600
-F 0 "U1" H 2600 3200 50  0000 C CNN
-F 1 "USB_PCB" H 2600 3300 50  0000 C CNN
+F 0 "U1" H 2600 4050 50  0000 C CNN
+F 1 "USB_PCB" H 2600 3950 50  0000 C CNN
 F 2 "footprint-lib.pretty:usb-PCB" H 2650 3650 50  0001 C CNN
 F 3 "" H 2650 3650 50  0001 C CNN
 	1    2650 3600
-	-1   0    0    1
-$EndComp
+	-1   0    0    -1
+$EndComp
+$Comp
+L customized_power:+5V #PWR0105
+U 1 1 5BC62F84
+P 3300 3300
+F 0 "#PWR0105" H 3300 3150 50  0001 C CNN
+F 1 "+5V" H 3350 3500 50  0000 C CNN
+F 2 "" H 3300 3300 50  0001 C CNN
+F 3 "" H 3300 3300 50  0001 C CNN
+	1    3300 3300
+	1    0    0    -1
+$EndComp
+Wire Wire Line
+	3300 3300 3300 3450
+Wire Wire Line
+	3300 3450 3000 3450
+$Comp
+L power:GND #PWR0106
+U 1 1 5BC63214
+P 3300 3900
+F 0 "#PWR0106" H 3300 3650 50  0001 C CNN
+F 1 "GND" H 3350 3700 50  0000 C CNN
+F 2 "" H 3300 3900 50  0001 C CNN
+F 3 "" H 3300 3900 50  0001 C CNN
+	1    3300 3900
+	1    0    0    -1
+$EndComp
+Wire Wire Line
+	3300 3900 3300 3750
+Wire Wire Line
+	3300 3750 3000 3750
+$Comp
+L customized_power:+5V #PWR0107
+U 1 1 5BC635B9
+P 2500 4700
+F 0 "#PWR0107" H 2500 4550 50  0001 C CNN
+F 1 "+5V" H 2550 4900 50  0000 C CNN
+F 2 "" H 2500 4700 50  0001 C CNN
+F 3 "" H 2500 4700 50  0001 C CNN
+	1    2500 4700
+	1    0    0    -1
+$EndComp
+$Comp
+L power:GND #PWR0108
+U 1 1 5BC635CE
+P 2500 5300
+F 0 "#PWR0108" H 2500 5050 50  0001 C CNN
+F 1 "GND" H 2550 5100 50  0000 C CNN
+F 2 "" H 2500 5300 50  0001 C CNN
+F 3 "" H 2500 5300 50  0001 C CNN
+	1    2500 5300
+	1    0    0    -1
+$EndComp
+$Comp
+L taobao-c:C106 C1
+U 1 1 5BC6366F
+P 2500 5000
+F 0 "C1" H 2600 5050 50  0000 L CNN
+F 1 "C106" H 2600 5000 50  0000 L CNN
+F 2 "Capacitor_SMD:C_0805_2012Metric_Pad1.15x1.40mm_HandSolder" H 2500 5000 50  0001 C CNN
+F 3 "~" H 2500 5000 50  0001 C CNN
+	1    2500 5000
+	1    0    0    -1
+$EndComp
+Wire Wire Line
+	2500 5100 2500 5300
+Wire Wire Line
+	2500 4700 2500 4900
+$Comp
+L customized_power:+5V #PWR0109
+U 1 1 5BC63CBF
+P 2950 4700
+F 0 "#PWR0109" H 2950 4550 50  0001 C CNN
+F 1 "+5V" H 3000 4900 50  0000 C CNN
+F 2 "" H 2950 4700 50  0001 C CNN
+F 3 "" H 2950 4700 50  0001 C CNN
+	1    2950 4700
+	1    0    0    -1
+$EndComp
+$Comp
+L taobao-r:R102 R3
+U 1 1 5BC63EB1
+P 2950 4900
+F 0 "R3" H 3050 4950 50  0000 L CNN
+F 1 "R102" H 3050 4900 50  0000 L CNN
+F 2 "Resistor_SMD:R_0805_2012Metric_Pad1.15x1.40mm_HandSolder" H 2950 4900 50  0001 C CNN
+F 3 "~" H 2950 4900 50  0001 C CNN
+	1    2950 4900
+	1    0    0    -1
+$EndComp
+$Comp
+L taobao-components:LED_GREEN D1
+U 1 1 5BC640C6
+P 2950 5200
+F 0 "D1" V 3000 5100 50  0000 R CNN
+F 1 "LED_GREEN" V 2950 5100 50  0000 R CNN
+F 2 "LED_SMD:LED_0805_2012Metric_Pad1.15x1.40mm_HandSolder" V 2950 5200 50  0001 C CNN
+F 3 "~" V 2950 5200 50  0001 C CNN
+	1    2950 5200
+	0    -1   -1   0
+$EndComp
+$Comp
+L power:GND #PWR0110
+U 1 1 5BC6417D
+P 2950 5400
+F 0 "#PWR0110" H 2950 5150 50  0001 C CNN
+F 1 "GND" H 3000 5200 50  0000 C CNN
+F 2 "" H 2950 5400 50  0001 C CNN
+F 3 "" H 2950 5400 50  0001 C CNN
+	1    2950 5400
+	1    0    0    -1
+$EndComp
+Wire Wire Line
+	2950 5300 2950 5400
+Wire Wire Line
+	2950 5000 2950 5100
+Wire Wire Line
+	2950 4700 2950 4800
+$Comp
+L taobao-r:R102 R4
+U 1 1 5BC65043
+P 3600 4900
+F 0 "R4" H 3700 4950 50  0000 L CNN
+F 1 "R102" H 3700 4900 50  0000 L CNN
+F 2 "Resistor_SMD:R_0805_2012Metric_Pad1.15x1.40mm_HandSolder" H 3600 4900 50  0001 C CNN
+F 3 "~" H 3600 4900 50  0001 C CNN
+	1    3600 4900
+	1    0    0    -1
+$EndComp
+$Comp
+L taobao-components:LED_GREEN D2
+U 1 1 5BC65049
+P 3600 5200
+F 0 "D2" V 3650 5100 50  0000 R CNN
+F 1 "LED_GREEN" V 3600 5100 50  0000 R CNN
+F 2 "LED_SMD:LED_0805_2012Metric_Pad1.15x1.40mm_HandSolder" V 3600 5200 50  0001 C CNN
+F 3 "~" V 3600 5200 50  0001 C CNN
+	1    3600 5200
+	0    -1   -1   0
+$EndComp
+$Comp
+L power:GND #PWR0111
+U 1 1 5BC6504F
+P 3600 5400
+F 0 "#PWR0111" H 3600 5150 50  0001 C CNN
+F 1 "GND" H 3650 5200 50  0000 C CNN
+F 2 "" H 3600 5400 50  0001 C CNN
+F 3 "" H 3600 5400 50  0001 C CNN
+	1    3600 5400
+	1    0    0    -1
+$EndComp
+Wire Wire Line
+	3600 5300 3600 5400
+Wire Wire Line
+	3600 5000 3600 5100
+Wire Wire Line
+	3600 4700 3600 4800
+$Comp
+L customized_power:+3V3 #PWR0112
+U 1 1 5BC655C0
+P 3600 4700
+F 0 "#PWR0112" H 3600 4550 50  0001 C CNN
+F 1 "+3V3" H 3650 4900 50  0000 C CNN
+F 2 "" H 3600 4700 50  0001 C CNN
+F 3 "" H 3600 4700 50  0001 C CNN
+	1    3600 4700
+	1    0    0    -1
+$EndComp
+$Sheet
+S 6400 3850 1200 750
+U 5BC671E5
+F0 "ESP8266" 50
+F1 "ESP8266.sch" 50
+$EndSheet
 $EndSCHEMATC

Commit message: update,
Parts:
- added U?: TPD2E001DRLR, Package_TO_SOT_SMD:SOT-23-5_HandSoldering, symbol taobao-components:TPD2E001DRLR
Connections:
- net +5V: now also U?.1 (VCC)
- net GND: now also U?.4 (GND)
- net at U1.2 (DM): now also U?.2 (NC), U?.5 (IO2)
- net at U1.3 (DP): now also U?.3 (IO1)
Other:
- moved on the sheet: U1
Changed lines of the file:
@@
 L taobao-components:USB_PCB U1
 U 1 1 5BC627DA
-P 2650 3600
-F 0 "U1" H 2600 4050 50  0000 C CNN
-F 1 "USB_PCB" H 2600 3950 50  0000 C CNN
-F 2 "footprint-lib.pretty:usb-PCB" H 2650 3650 50  0001 C CNN
-F 3 "" H 2650 3650 50  0001 C CNN
-	1    2650 3600
+P 7950 5750
+F 0 "U1" H 7900 6200 50  0000 C CNN
+F 1 "USB_PCB" H 7900 6100 50  0000 C CNN
+F 2 "footprint-lib.pretty:usb-PCB" H 7950 5800 50  0001 C CNN
+F 3 "" H 7950 5800 50  0001 C CNN
+	1    7950 5750
 	-1   0    0    -1
 $EndComp
@@
 L customized_power:+5V #PWR0105
 U 1 1 5BC62F84
-P 3300 3300
-F 0 "#PWR0105" H 3300 3150 50  0001 C CNN
-F 1 "+5V" H 3350 3500 50  0000 C CNN
-F 2 "" H 3300 3300 50  0001 C CNN
-F 3 "" H 3300 3300 50  0001 C CNN
-	1    3300 3300
-	1    0    0    -1
-$EndComp
-Wire Wire Line
-	3300 3300 3300 3450
-Wire Wire Line
-	3300 3450 3000 3450
+P 8600 5450
+F 0 "#PWR0105" H 8600 5300 50  0001 C CNN
+F 1 "+5V" H 8650 5650 50  0000 C CNN
+F 2 "" H 8600 5450 50  0001 C CNN
+F 3 "" H 8600 5450 50  0001 C CNN
+	1    8600 5450
+	1    0    0    -1
+$EndComp
+Wire Wire Line
+	8600 5450 8600 5600
+Wire Wire Line
+	8600 5600 8300 5600
 $Comp
 L power:GND #PWR0106
 U 1 1 5BC63214
-P 3300 3900
-F 0 "#PWR0106" H 3300 3650 50  0001 C CNN
-F 1 "GND" H 3350 3700 50  0000 C CNN
-F 2 "" H 3300 3900 50  0001 C CNN
-F 3 "" H 3300 3900 50  0001 C CNN
-	1    3300 3900
-	1    0    0    -1
-$EndComp
-Wire Wire Line
-	3300 3900 3300 3750
-Wire Wire Line
-	3300 3750 3000 3750
+P 8600 6050
+F 0 "#PWR0106" H 8600 5800 50  0001 C CNN
+F 1 "GND" H 8650 5850 50  0000 C CNN
+F 2 "" H 8600 6050 50  0001 C CNN
+F 3 "" H 8600 6050 50  0001 C CNN
+	1    8600 6050
+	1    0    0    -1
+$EndComp
+Wire Wire Line
+	8600 6050 8600 5900
+Wire Wire Line
+	8600 5900 8300 5900
 $Comp
 L customized_power:+5V #PWR0107
@@
 $EndComp
 $Sheet
-S 6400 3850 1200 750
+S 9350 2800 1200 750
 U 5BC671E5
 F0 "ESP8266" 50
 F1 "ESP8266.sch" 50
 $EndSheet
+$Comp
+L taobao-components:TPD2E001DRLR U?
+U 1 1 5BD8AA4C
+P 9900 5750
+F 0 "U?" H 9900 6350 60  0000 C CNN
+F 1 "TPD2E001DRLR" H 9900 6200 60  0000 C CNN
+F 2 "Package_TO_SOT_SMD:SOT-23-5_HandSoldering" H 9900 6100 60  0000 C CNN
+F 3 "" H 9900 5750 60  0000 C CNN
+	1    9900 5750
+	1    0    0    -1
+$EndComp
+Wire Wire Line
+	8300 5800 8900 5800
+Wire Wire Line
+	8900 5800 8900 5900
+Wire Wire Line
+	8900 5900 9350 5900
+Wire Wire Line
+	8300 5700 9100 5700
+Wire Wire Line
+	9100 5700 9100 5750
+Wire Wire Line
+	9100 5750 9350 5750
+Wire Wire Line
+	9100 5700 9100 5100
+Wire Wire Line
+	9100 5100 10600 5100
+Wire Wire Line
+	10600 5100 10600 5600
+Wire Wire Line
+	10600 5600 10450 5600
+Connection ~ 9100 5700
+$Comp
+L customized_power:+5V #PWR?
+U 1 1 5BD8C440
+P 9250 5450
+F 0 "#PWR?" H 9250 5300 50  0001 C CNN
+F 1 "+5V" H 9300 5650 50  0000 C CNN
+F 2 "" H 9250 5450 50  0001 C CNN
+F 3 "" H 9250 5450 50  0001 C CNN
+	1    9250 5450
+	1    0    0    -1
+$EndComp
+Wire Wire Line
+	9250 5450 9250 5600
+Wire Wire Line
+	9250 5600 9350 5600
+$Comp
+L power:GND #PWR?
+U 1 1 5BD8CD65
+P 10650 6050
+F 0 "#PWR?" H 10650 5800 50  0001 C CNN
+F 1 "GND" H 10700 5850 50  0000 C CNN
+F 2 "" H 10650 6050 50  0001 C CNN
+F 3 "" H 10650 6050 50  0001 C CNN
+	1    10650 6050
+	1    0    0    -1
+$EndComp
+Wire Wire Line
+	10450 5900 10650 5900
+Wire Wire Line
+	10650 5900 10650 6050
 $EndSCHEMATC

Commit message: update,
Parts:
- removed U1: USB_PCB, footprint-lib.pretty:usb-PCB, symbol taobao-components:USB_PCB
- removed U?: TPD2E001DRLR, Package_TO_SOT_SMD:SOT-23-5_HandSoldering, symbol taobao-components:TPD2E001DRLR
Other:
- moved on the sheet: C1, D1, D2, R3, R4

Commit message: update,
Parts:
- J2: footprint Connector_PinHeader_2.54mm:PinHeader_1x08_P2.54mm_Vertical -> footprint-lib:PMS5003S
Changed lines of the file:
@@
 F 0 "J2" H 3550 2300 50  0000 C CNN
 F 1 "CONN_PMS" H 3550 2200 50  0000 C CNN
-F 2 "Connector_PinHeader_2.54mm:PinHeader_1x08_P2.54mm_Vertical" H 3650 1750 50  0001 C CNN
+F 2 "footprint-lib:PMS5003S" H 3650 1750 50  0001 C CNN
 F 3 "~" H 3650 1750 50  0001 C CNN
 	1    3650 1750
